File: hardware/sdiskII_stm32.kicad_pcb (KiCad board)
At the start: 2 copper layers, 76 x 56.3 mm, 17 parts, among them J1 PWR, J2 APPLE_SDISKII, J3 Conn_01x06, J4 UART, J6 STLINK, U2 MicroSD_SDIO, U8 DM-OLED096-636

Commit message: pcb small change v5
Parts:
- removed DEBUG: Conn_01x04, Connector_PinHeader_2.54mm:PinHeader_1x04_P2.54mm_Vertical
- added D1: 1N4148, Diode_THT:D_DO-35_SOD27_P7.62mm_Horizontal, F.Cu at (205.0, 114.8)
- added G***: LOGO, Stm32F411:snap, F.Cu at (177.0, 114.9)
- added J5: Conn_01x04, Connector_PinHeader_2.54mm:PinHeader_1x04_P2.54mm_Vertical, F.Cu at (134.9, 116.4)
- moved J3 5.86 mm to (205.0, 118.9)
- moved JP1 0.32 mm to (205.0, 104.7)
Connections:
- J1 pad 2: PWR_IN -> PWR_RD
- JP1 pad 1: PWR_IN -> PWR_RD
- U2 pad : (no net) -> GND
- U2 pad ~: GND -> (no net)
Routing:
- net GND: track 243.5 -> 264.7 mm, vias 2 -> 3
- net PWR_IN: track 110.2 -> 118.9 mm
- net PWR_RD: track 0.00 -> 6.97 mm
- net WR_DATA: track 82.4 -> 88.3 mm
- net WR_REQ: track 116.1 -> 121.9 mm
- net RD_DATA: track 70.8 -> 76.5 mm
- net WR_PROTECT: track 67.2 -> 72.6 mm
- net DEVICE_ENABLE: track 89.8 -> 95.1 mm
Other:
- board text added: "SMARTDISK II REV.5"
- board text removed: "SMARTDISK II REV.4"

Commit message: v0.80.12 beta
Parts:
- added D2: 1N4148WT, Diode_SMD:D_0805_2012Metric_Pad1.15x1.40mm_HandSolder, F.Cu at (205.0, 110.8)
- added R4: 330, Resistor_SMD:R_0805_2012Metric_Pad1.20x1.40mm_HandSolder, B.Cu at (157.8, 126.5)
- added R5: 330, Resistor_SMD:R_0805_2012Metric_Pad1.20x1.40mm_HandSolder, B.Cu at (157.8, 106.1)
Connections:
- J2 pad 12: SELECT -> SELECT_D
- J2 pad 7: 3.5DSK -> 3.5DSK_D
- U2 pad : GND -> (no net)
Routing:
- net SELECT: track 73.8 -> 2.80 mm, vias 1 -> 0
- net SELECT_D: track 0.00 -> 69.0 mm, vias 0 -> 1
- net 3.5DSK_D: track 0.00 -> 41.5 mm
- net 3.5DSK: track 43.1 -> 2.67 mm
- net PWR_IN: track 118.9 -> 121.9 mm
- net PWR_RD: track 6.97 -> 9.38 mm
Other:
- board text added: "SMARTDISK II REV.6"
- board text removed: "SMARTDISK II REV.5"

Commit message: PCB Rev6
Parts:
- added D3: 1N4148WT, Diode_SMD:D_0805_2012Metric_Pad1.15x1.40mm_HandSolder, F.Cu at (201.5, 110.8)
Connections:
- μC1 pad 9: unconnected-(μC1-A12-Pad9) -> A2PWR
Routing:
- net A2PWR: track 0.00 -> 49.8 mm, vias 0 -> 5
- net GND: track 264.7 -> 272.6 mm, vias 3 -> 4
- net VCC: track 24.4 -> 30.7 mm
Other:
- board text added: "REV6: (beta) - Adding A2PWR PA12, Apple II PWR check on external PWR supply - Adding D3, to avoid PA12 -> Apple PWR supply REV5: (beta) - Adding D1 & D2 protection (only one is needed), - Adding more GND to SDCARD - Adding R4 PIN SELECT for protection on DISK3.5 use - Adding R5 PIN SELECT for protection on DISK3.5 use REV4: (Last production & tested version) - Adding PWR pads - Moving SDCard"
